File: Board/board.sch (EAGLE design)
At the start: 49 parts, among them IC1 L297, IC2 MEGA32-P, IC3 L298, J1 +12V, Q1 BC639, Q3 BC639, U1 MCP9808MSOP, X1 WATER_PUMP, X2 FAN, X5 SM_CD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

Commit message: auto route
Parts:
- VSS_LED: device led:LED3MM -> led:LED5MM
Connections:
- net GND: now also VSS_LED.C; no longer R3.1
- net N$7: now also R3.1, VSS_LED.A; no longer R3.2, VSS_LED.C
- net VSS: now also R3.2; no longer VSS_LED.A
Other:
- moved on the sheet: R3, VSS_LED
Changed lines of the file:
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@@
 <part name="C11" library="rcl" deviceset="C-EU" device="025-025X050" value="100nF"/>
 <part name="SUPPLY29" library="supply2" deviceset="GND" device=""/>
-<part name="VSS_LED" library="led" deviceset="LED" device="3MM"/>
 <part name="R3" library="rcl" deviceset="R-EU_" device="0207/12" value="470R"/>
 <part name="SUPPLY30" library="supply2" deviceset="GND" device=""/>
@@
 <part name="FAN_LED" library="led" deviceset="LED" device="5MM"/>
 <part name="CTRL_LED" library="led" deviceset="LED" device="5MM"/>
+<part name="VSS_LED" library="led" deviceset="LED" device="5MM"/>
 </parts>
 <sheets>
@@
 <instance part="C11" gate="G$1" x="-73.66" y="-99.06"/>
 <instance part="SUPPLY29" gate="GND" x="-73.66" y="-109.22"/>
-<instance part="VSS_LED" gate="G$1" x="-45.72" y="134.62"/>
-<instance part="R3" gate="G$1" x="-45.72" y="116.84" rot="R90"/>
+<instance part="R3" gate="G$1" x="-45.72" y="129.54" rot="R90"/>
 <instance part="SUPPLY30" gate="GND" x="-45.72" y="104.14"/>
 <instance part="WP_LED" gate="G$1" x="457.2" y="-132.08"/>
 <instance part="FAN_LED" gate="G$1" x="457.2" y="-30.48"/>
 <instance part="CTRL_LED" gate="G$1" x="12.7" y="-27.94"/>
+<instance part="VSS_LED" gate="G$1" x="-45.72" y="116.84"/>
 </instances>
 <busses>
@@
 <junction x="-58.42" y="142.24"/>
 <wire x1="-58.42" y1="142.24" x2="-45.72" y2="142.24" width="0.1524" layer="91"/>
-<pinref part="VSS_LED" gate="G$1" pin="A"/>
-<wire x1="-45.72" y1="142.24" x2="-45.72" y2="137.16" width="0.1524" layer="91"/>
+<pinref part="R3" gate="G$1" pin="2"/>
+<wire x1="-45.72" y1="142.24" x2="-45.72" y2="134.62" width="0.1524" layer="91"/>
 </segment>
 <segment>
@@
 </segment>
 <segment>
-<pinref part="SUPPLY30" gate="GND" pin="GND"/>
-<pinref part="R3" gate="G$1" pin="1"/>
-<wire x1="-45.72" y1="106.68" x2="-45.72" y2="111.76" width="0.1524" layer="91"/>
-</segment>
-<segment>
 <pinref part="WP_LED" gate="G$1" pin="C"/>
 <pinref part="SUPPLY22" gate="GND" pin="GND"/>
@@
 <pinref part="SUPPLY25" gate="GND" pin="GND"/>
 <wire x1="12.7" y1="-33.02" x2="12.7" y2="-40.64" width="0.1524" layer="91"/>
+</segment>
+<segment>
+<pinref part="VSS_LED" gate="G$1" pin="C"/>
+<pinref part="SUPPLY30" gate="GND" pin="GND"/>
+<wire x1="-45.72" y1="111.76" x2="-45.72" y2="106.68" width="0.1524" layer="91"/>
 </segment>
 </net>
@@
 </segment>
 </net>
-<net name="N$7" class="0">
-<segment>
-<pinref part="R3" gate="G$1" pin="2"/>
-<pinref part="VSS_LED" gate="G$1" pin="C"/>
-<wire x1="-45.72" y1="121.92" x2="-45.72" y2="129.54" width="0.1524" layer="91"/>
-</segment>
-</net>
 <net name="N$11" class="0">
 <segment>
@@
 </segment>
 </net>
+<net name="N$7" class="0">
+<segment>
+<pinref part="R3" gate="G$1" pin="1"/>
+<pinref part="VSS_LED" gate="G$1" pin="A"/>
+<wire x1="-45.72" y1="124.46" x2="-45.72" y2="119.38" width="0.1524" layer="91"/>
+</segment>
+</net>

Commit message: added 5mm vss led
Parts:
- R1, R5: value (none) -> 220R
Connections:
- removed net VSS1: D10.C, D3.A, D4.A, D6.A, D7.C, D8.C, IC3.OUT1, IC3.OUT2, IC3.OUT4, X5-1.KL, X6-1.KL, X6-2.KL
- new net N$24: D10.C, D6.A, IC3.OUT4, X5-1.KL
- new net N$25: D3.A, D7.C, IC3.OUT1, X6-2.KL
- net GND: now also IC2.AGND
- net N$26: now also D4.A, D8.C, IC3.OUT2, X6-1.KL; no longer IC2.(AIN0/INT2)PB2
- net VCC: now also IC2.AREF
Changed lines of the file:
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@@
 <part name="X2" library="con-ptr500" deviceset="AK500/3" device="" value="FAN"/>
 <part name="SUPPLY11" library="supply2" deviceset="GND" device=""/>
-<part name="R1" library="rcl" deviceset="R-EU_" device="0207/12"/>
+<part name="R1" library="rcl" deviceset="R-EU_" device="0207/12" value="220R"/>
 <part name="VSS4" library="supply1" deviceset="VSS" device=""/>
 <part name="Q1" library="transistor-small-signal" deviceset="BC639" device=""/>
@@
 <part name="D2" library="diode" deviceset="1N581*" device="" technology="9-B" value="1N5824"/>
 <part name="SUPPLY20" library="supply2" deviceset="GND" device=""/>
-<part name="R5" library="rcl" deviceset="R-EU_" device="0207/12"/>
+<part name="R5" library="rcl" deviceset="R-EU_" device="0207/12" value="220R"/>
 <part name="VSS6" library="supply1" deviceset="VSS" device=""/>
 <part name="Q3" library="transistor-small-signal" deviceset="BC639" device=""/>
@@
 <wire x1="-76.2" y1="22.86" x2="-81.28" y2="22.86" width="0.1524" layer="91"/>
 <wire x1="-81.28" y1="22.86" x2="-81.28" y2="15.24" width="0.1524" layer="91"/>
+<pinref part="IC2" gate="G$1" pin="AGND"/>
+<wire x1="-76.2" y1="30.48" x2="-81.28" y2="30.48" width="0.1524" layer="91"/>
+<wire x1="-81.28" y1="30.48" x2="-81.28" y2="22.86" width="0.1524" layer="91"/>
+<junction x="-81.28" y="22.86"/>
 </segment>
 <segment>
@@
 <pinref part="P+3" gate="VCC" pin="VCC"/>
 <wire x1="-76.2" y1="25.4" x2="-88.9" y2="25.4" width="0.1524" layer="91"/>
-<wire x1="-88.9" y1="25.4" x2="-88.9" y2="40.64" width="0.1524" layer="91"/>
+<wire x1="-88.9" y1="25.4" x2="-88.9" y2="35.56" width="0.1524" layer="91"/>
 <pinref part="C4" gate="G$1" pin="1"/>
+<wire x1="-88.9" y1="35.56" x2="-88.9" y2="40.64" width="0.1524" layer="91"/>
 <wire x1="-88.9" y1="25.4" x2="-88.9" y2="22.86" width="0.1524" layer="91"/>
 <junction x="-88.9" y="25.4"/>
+<pinref part="IC2" gate="G$1" pin="AREF"/>
+<wire x1="-76.2" y1="35.56" x2="-88.9" y2="35.56" width="0.1524" layer="91"/>
+<junction x="-88.9" y="35.56"/>
 </segment>
 <segment>
@@
 </segment>
 </net>
-<net name="N$26" class="0">
-<segment>
-<pinref part="IC2" gate="G$1" pin="(AIN0/INT2)PB2"/>
-<wire x1="-35.56" y1="17.78" x2="12.7" y2="17.78" width="0.1524" layer="91"/>
-</segment>
-</net>
 <net name="N$35" class="0">
 <segment>
@@
 </segment>
 </net>
-<net name="VSS1" class="0">
-<segment>
-<pinref part="D8" gate="G$1" pin="C"/>
-<pinref part="X6" gate="-1" pin="KL"/>
-<wire x1="307.34" y1="-160.02" x2="325.12" y2="-160.02" width="0.1524" layer="91"/>
-<wire x1="307.34" y1="-167.64" x2="307.34" y2="-160.02" width="0.1524" layer="91"/>
-<wire x1="274.32" y1="-167.64" x2="307.34" y2="-167.64" width="0.1524" layer="91"/>
-<pinref part="D4" gate="G$1" pin="A"/>
-<wire x1="274.32" y1="-149.86" x2="274.32" y2="-167.64" width="0.1524" layer="91"/>
-<junction x="274.32" y="-167.64"/>
-<wire x1="274.32" y1="-167.64" x2="274.32" y2="-185.42" width="0.1524" layer="91"/>
-<pinref part="IC3" gate="L298" pin="OUT2"/>
-<wire x1="251.46" y1="-167.64" x2="274.32" y2="-167.64" width="0.1524" layer="91"/>
-</segment>
-<segment>
-<pinref part="X5" gate="-1" pin="KL"/>
-<pinref part="D10" gate="G$1" pin="C"/>
-<wire x1="294.64" y1="-172.72" x2="294.64" y2="-185.42" width="0.1524" layer="91"/>
-<wire x1="294.64" y1="-172.72" x2="325.12" y2="-172.72" width="0.1524" layer="91"/>
-<junction x="294.64" y="-172.72"/>
-<pinref part="IC3" gate="L298" pin="OUT4"/>
-<wire x1="251.46" y1="-172.72" x2="294.64" y2="-172.72" width="0.1524" layer="91"/>
-<pinref part="D6" gate="G$1" pin="A"/>
-<wire x1="294.64" y1="-149.86" x2="294.64" y2="-172.72" width="0.1524" layer="91"/>
-</segment>
-<segment>
-<pinref part="D7" gate="G$1" pin="C"/>
-<pinref part="IC3" gate="L298" pin="OUT1"/>
-<wire x1="251.46" y1="-165.1" x2="264.16" y2="-165.1" width="0.1524" layer="91"/>
-<wire x1="264.16" y1="-165.1" x2="304.8" y2="-165.1" width="0.1524" layer="91"/>
-<wire x1="304.8" y1="-165.1" x2="304.8" y2="-154.94" width="0.1524" layer="91"/>
-<pinref part="X6" gate="-2" pin="KL"/>
-<wire x1="304.8" y1="-154.94" x2="325.12" y2="-154.94" width="0.1524" layer="91"/>
-<pinref part="D3" gate="G$1" pin="A"/>
-<wire x1="264.16" y1="-149.86" x2="264.16" y2="-165.1" width="0.1524" layer="91"/>
-<junction x="264.16" y="-165.1"/>
-<wire x1="264.16" y1="-165.1" x2="264.16" y2="-185.42" width="0.1524" layer="91"/>
-</segment>
-</net>
 <net name="N$11" class="0">
 <segment>
@@
 </segment>
 </net>
-<net name="N$24" class="0">
-<segment>
-<pinref part="D9" gate="G$1" pin="C"/>
+<net name="N$7" class="0">
+<segment>
+<pinref part="R3" gate="G$1" pin="1"/>
+<pinref part="VSS_LED" gate="G$1" pin="A"/>
+<wire x1="-45.72" y1="124.46" x2="-45.72" y2="119.38" width="0.1524" layer="91"/>
+</segment>
+</net>
+<net name="N$25" class="0">
+<segment>
+<pinref part="X6" gate="-2" pin="KL"/>
+<wire x1="304.8" y1="-154.94" x2="325.12" y2="-154.94" width="0.1524" layer="91"/>
+<wire x1="304.8" y1="-165.1" x2="304.8" y2="-154.94" width="0.1524" layer="91"/>
+<pinref part="IC3" gate="L298" pin="OUT1"/>
+<wire x1="251.46" y1="-165.1" x2="264.16" y2="-165.1" width="0.1524" layer="91"/>
+<pinref part="D3" gate="G$1" pin="A"/>
+<wire x1="264.16" y1="-165.1" x2="304.8" y2="-165.1" width="0.1524" layer="91"/>
+<wire x1="264.16" y1="-149.86" x2="264.16" y2="-165.1" width="0.1524" layer="91"/>
+<junction x="264.16" y="-165.1"/>
+<pinref part="D7" gate="G$1" pin="C"/>
+<wire x1="264.16" y1="-165.1" x2="264.16" y2="-185.42" width="0.1524" layer="91"/>
+</segment>
+</net>
+<net name="N$26" class="0">
+<segment>
+<pinref part="X6" gate="-1" pin="KL"/>
+<wire x1="307.34" y1="-160.02" x2="325.12" y2="-160.02" width="0.1524" layer="91"/>
+<wire x1="307.34" y1="-167.64" x2="307.34" y2="-160.02" width="0.1524" layer="91"/>
+<pinref part="IC3" gate="L298" pin="OUT2"/>
+<wire x1="307.34" y1="-167.64" x2="274.32" y2="-167.64" width="0.1524" layer="91"/>
+<pinref part="D4" gate="G$1" pin="A"/>
+<wire x1="274.32" y1="-167.64" x2="251.46" y2="-167.64" width="0.1524" layer="91"/>
+<wire x1="274.32" y1="-149.86" x2="274.32" y2="-167.64" width="0.1524" layer="91"/>
+<junction x="274.32" y="-167.64"/>
+<wire x1="274.32" y1="-167.64" x2="274.32" y2="-185.42" width="0.1524" layer="91"/>
+<pinref part="D8" gate="G$1" pin="C"/>
+</segment>
+</net>
+<net name="N$27" class="0">
+<segment>
 <pinref part="X5" gate="-2" pin="KL"/>
 <wire x1="309.88" y1="-167.64" x2="325.12" y2="-167.64" width="0.1524" layer="91"/>
 <wire x1="309.88" y1="-170.18" x2="309.88" y2="-167.64" width="0.1524" layer="91"/>
+<pinref part="IC3" gate="L298" pin="OUT3"/>
+<wire x1="251.46" y1="-170.18" x2="284.48" y2="-170.18" width="0.1524" layer="91"/>
+<pinref part="D5" gate="G$1" pin="A"/>
 <wire x1="284.48" y1="-170.18" x2="309.88" y2="-170.18" width="0.1524" layer="91"/>
-<pinref part="D5" gate="G$1" pin="A"/>
 <wire x1="284.48" y1="-149.86" x2="284.48" y2="-170.18" width="0.1524" layer="91"/>
 <junction x="284.48" y="-170.18"/>
+<pinref part="D9" gate="G$1" pin="C"/>
 <wire x1="284.48" y1="-170.18" x2="284.48" y2="-185.42" width="0.1524" layer="91"/>
-<pinref part="IC3" gate="L298" pin="OUT3"/>
-<wire x1="251.46" y1="-170.18" x2="284.48" y2="-170.18" width="0.1524" layer="91"/>
-</segment>
-</net>
-<net name="N$7" class="0">
-<segment>
-<pinref part="R3" gate="G$1" pin="1"/>
-<pinref part="VSS_LED" gate="G$1" pin="A"/>
-<wire x1="-45.72" y1="124.46" x2="-45.72" y2="119.38" width="0.1524" layer="91"/>
+</segment>
+</net>
+<net name="N$24" class="0">
+<segment>
+<pinref part="IC3" gate="L298" pin="OUT4"/>
+<pinref part="X5" gate="-1" pin="KL"/>
+<wire x1="251.46" y1="-172.72" x2="294.64" y2="-172.72" width="0.1524" layer="91"/>
+<pinref part="D6" gate="G$1" pin="A"/>
+<wire x1="294.64" y1="-172.72" x2="325.12" y2="-172.72" width="0.1524" layer="91"/>
+<wire x1="294.64" y1="-149.86" x2="294.64" y2="-172.72" width="0.1524" layer="91"/>
+<junction x="294.64" y="-172.72"/>
+<pinref part="D10" gate="G$1" pin="C"/>
+<wire x1="294.64" y1="-172.72" x2="294.64" y2="-185.42" width="0.1524" layer="91"/>
 </segment>
 </net>
@@
 </sheet>
 </sheets>
+<errors>
+</errors>
 </schematic>
 </drawing>

Commit message: ds
Parts:
- removed U1: MCP9808MSOP, MCP9808:MCP9808MSOP
- added R6, R8: 4K7, rcl:R-EU_0207/12
- added U2: DS1621+, ds1621p:DS1621+
Connections:
- net GND: now also U2.A0, U2.A1, U2.A2, U2.GND; no longer U1.A0, U1.A1, U1.A2, U1.GND
- net N$35: now also R8.1, U2.SCL; no longer U1.SDA
- net N$36: now also R6.1, U2.SDA; no longer U1.SCL
- net VCC: now also R6.2, R8.2, U2.VDD; no longer U1.VDD
Other:
- moved on the sheet: C8
Changed lines of the file:
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@@
 <setting verticaltext="up"/>
 </settings>
-<grid distance="0.1" unitdist="inch" unit="inch" style="dots" multiple="1" display="yes" altdistance="0.01" altunitdist="inch" altunit="inch"/>
+<grid distance="0.1" unitdist="inch" unit="inch" style="lines" multiple="1" display="no" altdistance="0.01" altunitdist="inch" altunit="inch"/>
 <layers>
 <layer number="1" name="Top" color="4" fill="1" visible="no" active="no"/>
@@
 <part name="R12" library="rcl" deviceset="R-EU_" device="0207/12" value="330R"/>
 <part name="SUPPLY25" library="supply2" deviceset="GND" device=""/>
-<part name="U1" library="MCP9808" deviceset="MCP9808" device="MSOP"/>
 <part name="SUPPLY26" library="supply2" deviceset="GND" device=""/>
 <part name="C8" library="rcl" deviceset="C-EU" device="025-025X050" value="100nF"/>
@@
 <part name="CTRL_LED" library="led" deviceset="LED" device="5MM"/>
 <part name="VSS_LED" library="led" deviceset="LED" device="5MM"/>
+<part name="U2" library="ds1621p" deviceset="DS1621+" device=""/>
+<part name="SUPPLY31" library="supply2" deviceset="GND" device=""/>
+<part name="R6" library="rcl" deviceset="R-EU_" device="0207/12" value="4K7"/>
+<part name="R8" library="rcl" deviceset="R-EU_" device="0207/12" value="4K7"/>
+<part name="P+8" library="supply1" deviceset="VCC" device=""/>
+<part name="P+9" library="supply1" deviceset="VCC" device=""/>
 </parts>
 <sheets>
@@
 <instance part="R12" gate="G$1" x="12.7" y="-10.16" rot="R90"/>
 <instance part="SUPPLY25" gate="GND" x="12.7" y="-43.18"/>
-<instance part="U1" gate="G$1" x="-127" y="-132.08"/>
-<instance part="SUPPLY26" gate="GND" x="-147.32" y="-147.32"/>
-<instance part="C8" gate="G$1" x="-157.48" y="-134.62"/>
-<instance part="SUPPLY27" gate="GND" x="-157.48" y="-147.32"/>
-<instance part="P+14" gate="VCC" x="-157.48" y="-111.76"/>
+<instance part="SUPPLY26" gate="GND" x="-167.64" y="-147.32"/>
+<instance part="C8" gate="G$1" x="-185.42" y="-134.62"/>
+<instance part="SUPPLY27" gate="GND" x="-185.42" y="-147.32"/>
+<instance part="P+14" gate="VCC" x="-185.42" y="-111.76"/>
 <instance part="IC3" gate="L298" x="236.22" y="-167.64"/>
 <instance part="SUPPLY17" gate="GND" x="215.9" y="-198.12"/>
@@
 <instance part="CTRL_LED" gate="G$1" x="12.7" y="-27.94"/>
 <instance part="VSS_LED" gate="G$1" x="-45.72" y="116.84"/>
+<instance part="U2" gate="A" x="-109.22" y="-127" rot="R180"/>
+<instance part="SUPPLY31" gate="GND" x="-104.14" y="-147.32"/>
+<instance part="R6" gate="G$1" x="-160.02" y="-78.74" rot="R90"/>
+<instance part="R8" gate="G$1" x="-149.86" y="-78.74" rot="R90"/>
+<instance part="P+8" gate="VCC" x="-160.02" y="-60.96"/>
+<instance part="P+9" gate="VCC" x="-149.86" y="-60.96"/>
 </instances>
 <busses>
@@
 </segment>
 <segment>
-<pinref part="U1" gate="G$1" pin="GND"/>
-<wire x1="-142.24" y1="-139.7" x2="-147.32" y2="-139.7" width="0.1524" layer="91"/>
 <pinref part="SUPPLY26" gate="GND" pin="GND"/>
-<wire x1="-147.32" y1="-139.7" x2="-147.32" y2="-144.78" width="0.1524" layer="91"/>
-<pinref part="U1" gate="G$1" pin="A2"/>
-<wire x1="-142.24" y1="-134.62" x2="-147.32" y2="-134.62" width="0.1524" layer="91"/>
-<wire x1="-147.32" y1="-134.62" x2="-147.32" y2="-139.7" width="0.1524" layer="91"/>
-<junction x="-147.32" y="-139.7"/>
-<pinref part="U1" gate="G$1" pin="A1"/>
-<wire x1="-142.24" y1="-132.08" x2="-147.32" y2="-132.08" width="0.1524" layer="91"/>
-<wire x1="-147.32" y1="-132.08" x2="-147.32" y2="-134.62" width="0.1524" layer="91"/>
-<junction x="-147.32" y="-134.62"/>
-<pinref part="U1" gate="G$1" pin="A0"/>
-<wire x1="-142.24" y1="-129.54" x2="-147.32" y2="-129.54" width="0.1524" layer="91"/>
-<wire x1="-147.32" y1="-129.54" x2="-147.32" y2="-132.08" width="0.1524" layer="91"/>
-<junction x="-147.32" y="-132.08"/>
+<wire x1="-167.64" y1="-119.38" x2="-167.64" y2="-121.92" width="0.1524" layer="91"/>
+<pinref part="U2" gate="A" pin="A2"/>
+<wire x1="-167.64" y1="-121.92" x2="-167.64" y2="-124.46" width="0.1524" layer="91"/>
+<wire x1="-167.64" y1="-124.46" x2="-167.64" y2="-144.78" width="0.1524" layer="91"/>
+<wire x1="-167.64" y1="-119.38" x2="-162.56" y2="-119.38" width="0.1524" layer="91"/>
+<pinref part="U2" gate="A" pin="A1"/>
+<wire x1="-167.64" y1="-121.92" x2="-162.56" y2="-121.92" width="0.1524" layer="91"/>
+<junction x="-167.64" y="-121.92"/>
+<pinref part="U2" gate="A" pin="A0"/>
+<wire x1="-167.64" y1="-124.46" x2="-162.56" y2="-124.46" width="0.1524" layer="91"/>
+<junction x="-167.64" y="-124.46"/>
 </segment>
 <segment>
 <pinref part="C8" gate="G$1" pin="2"/>
 <pinref part="SUPPLY27" gate="GND" pin="GND"/>
-<wire x1="-157.48" y1="-139.7" x2="-157.48" y2="-144.78" width="0.1524" layer="91"/>
+<wire x1="-185.42" y1="-139.7" x2="-185.42" y2="-144.78" width="0.1524" layer="91"/>
 </segment>
 <segment>
@@
 <pinref part="SUPPLY30" gate="GND" pin="GND"/>
 <wire x1="-45.72" y1="111.76" x2="-45.72" y2="106.68" width="0.1524" layer="91"/>
+</segment>
+<segment>
+<pinref part="U2" gate="A" pin="GND"/>
+<wire x1="-111.76" y1="-119.38" x2="-104.14" y2="-119.38" width="0.1524" layer="91"/>
+<pinref part="SUPPLY31" gate="GND" pin="GND"/>
+<wire x1="-104.14" y1="-119.38" x2="-104.14" y2="-144.78" width="0.1524" layer="91"/>
 </segment>
 </net>
@@
 </segment>
 <segment>
-<pinref part="U1" gate="G$1" pin="VDD"/>
-<wire x1="-142.24" y1="-124.46" x2="-157.48" y2="-124.46" width="0.1524" layer="91"/>
 <pinref part="C8" gate="G$1" pin="1"/>
-<wire x1="-157.48" y1="-124.46" x2="-157.48" y2="-132.08" width="0.1524" layer="91"/>
 <pinref part="P+14" gate="VCC" pin="VCC"/>
-<wire x1="-157.48" y1="-114.3" x2="-157.48" y2="-124.46" width="0.1524" layer="91"/>
-<junction x="-157.48" y="-124.46"/>
+<wire x1="-185.42" y1="-114.3" x2="-185.42" y2="-127" width="0.1524" layer="91"/>
+<pinref part="U2" gate="A" pin="VDD"/>
+<wire x1="-185.42" y1="-127" x2="-185.42" y2="-132.08" width="0.1524" layer="91"/>
+<wire x1="-162.56" y1="-127" x2="-185.42" y2="-127" width="0.1524" layer="91"/>
+<junction x="-185.42" y="-127"/>
 </segment>
 <segment>
@@
 <wire x1="-73.66" y1="-93.98" x2="-73.66" y2="-96.52" width="0.1524" layer="91"/>
 <junction x="-73.66" y="-93.98"/>
+</segment>
+<segment>
+<pinref part="P+8" gate="VCC" pin="VCC"/>
+<pinref part="R6" gate="G$1" pin="2"/>
+<wire x1="-160.02" y1="-63.5" x2="-160.02" y2="-73.66" width="0.1524" layer="91"/>
+</segment>
+<segment>
+<pinref part="P+9" gate="VCC" pin="VCC"/>
+<pinref part="R8" gate="G$1" pin="2"/>
+<wire x1="-149.86" y1="-63.5" x2="-149.86" y2="-73.66" width="0.1524" layer="91"/>
 </segment>
 </net>
@@
 <wire x1="-83.82" y1="-86.36" x2="-111.76" y2="-86.36" width="0.1524" layer="91"/>
 <wire x1="-83.82" y1="-55.88" x2="-83.82" y2="-86.36" width="0.1524" layer="91"/>
-<pinref part="U1" gate="G$1" pin="SDA"/>
-<wire x1="-83.82" y1="-86.36" x2="-83.82" y2="-124.46" width="0.1524" layer="91"/>
+<wire x1="-83.82" y1="-86.36" x2="-83.82" y2="-104.14" width="0.1524" layer="91"/>
+<junction x="-83.82" y="-86.36"/>
+<pinref part="U2" gate="A" pin="SCL"/>
+<wire x1="-83.82" y1="-104.14" x2="-83.82" y2="-124.46" width="0.1524" layer="91"/>
 <wire x1="-83.82" y1="-124.46" x2="-111.76" y2="-124.46" width="0.1524" layer="91"/>
-<junction x="-83.82" y="-86.36"/>
+<pinref part="R8" gate="G$1" pin="1"/>
+<wire x1="-83.82" y1="-104.14" x2="-149.86" y2="-104.14" width="0.1524" layer="91"/>
+<wire x1="-149.86" y1="-104.14" x2="-149.86" y2="-83.82" width="0.1524" layer="91"/>
+<junction x="-83.82" y="-104.14"/>
 </segment>
 </net>
@@
 <wire x1="-86.36" y1="-53.34" x2="-86.36" y2="-83.82" width="0.1524" layer="91"/>
 <wire x1="-86.36" y1="-83.82" x2="-111.76" y2="-83.82" width="0.1524" layer="91"/>
-<wire x1="-86.36" y1="-83.82" x2="-86.36" y2="-127" width="0.1524" layer="91"/>
+<wire x1="-86.36" y1="-83.82" x2="-86.36" y2="-101.6" width="0.1524" layer="91"/>
 <junction x="-86.36" y="-83.82"/>
-<pinref part="U1" gate="G$1" pin="SCL"/>
+<pinref part="U2" gate="A" pin="SDA"/>
+<wire x1="-86.36" y1="-101.6" x2="-86.36" y2="-127" width="0.1524" layer="91"/>
 <wire x1="-86.36" y1="-127" x2="-111.76" y2="-127" width="0.1524" layer="91"/>
-</segment>
-</net>
+<pinref part="R6" gate="G$1" pin="1"/>
+<wire x1="-86.36" y1="-101.6" x2="-160.02" y2="-101.6" width="0.1524" layer="91"/>
+<wire x1="-160.02" y1="-101.6" x2="-160.02" y2="-83.82" width="0.1524" layer="91"/>
+<junction x="-86.36" y="-101.6"/>
+</segment>
+</net>
